File: 12AU7-Amplifier.sch (KiCad schematic (older format))
At the start: 30 parts

Commit message: annotate schematic and add power flags
Parts:
- gave numbers to parts that had none: 28
Connections:
- wire segments 113 -> 118
Other:
- moved on the sheet: D1, R1

Commit message: Assign footprints, create Alps 100KAX2 lib
Parts:
- C1, C2: footprint (none) -> Capacitor_THT:C_Radial_D5.0mm_H11.0mm_P2.00mm; symbol Device:CP -> Device:C
- C3, C4: footprint (none) -> Capacitor_THT:CP_Radial_D8.0mm_P2.50mm
- C5, C6: footprint (none) -> Capacitor_THT:CP_Radial_D10.0mm_P5.00mm
- D1: footprint (none) -> LED_THT:LED_D5.0mm_Horizontal_O1.27mm_Z3.0mm
- J1, J3: footprint (none) -> digikey-footprints:Headphone_Jack_2.5mm_SJ1-3523N
- J2: footprint (none) -> Connector_BarrelJack:BarrelJack_Horizontal
- R1, R2, R3, R6, R7, R8, R9: footprint (none) -> Resistor_THT:R_Axial_DIN0207_L6.3mm_D2.5mm_P10.16mm_Horizontal
- R4, R5: footprint (none) -> Resistor_THT:R_Axial_DIN0614_L14.3mm_D5.7mm_P5.08mm_Vertical
- RV1: value 50kΩ -> 100kΩ; footprint (none) -> Alps_100KAX2:Alps_100KAX2
- RV2, RV3: footprint (none) -> Potentiometer_THT:Potentiometer_Piher_PT-10-H01_Horizontal
- SW1: footprint (none) -> digikey-footprints:Toggle_Switch_100SP1T1B4M2QE
- U2, U3: footprint (none) -> Package_TO_SOT_THT:TO-220-3_Vertical
Connections:
- wire segments 118 -> 121
Other:
- moved on the sheet: J3
Changed lines of the file:
@@
 F 0 "J1" H 1782 3725 50  0000 C CNN
 F 1 "AudioIn" H 1782 3634 50  0000 C CNN
-F 2 "" H 1800 3400 50  0001 C CNN
+F 2 "digikey-footprints:Headphone_Jack_2.5mm_SJ1-3523N" H 1800 3400 50  0001 C CNN
 F 3 "~" H 1800 3400 50  0001 C CNN
 	1    1800 3400
 	1    0    0    -1
 $EndComp
-$Comp
-L Device:R_POT_Dual RV1
-U 1 1 5CAAC98A
-P 2750 3450
-F 0 "RV1" V 2704 3263 50  0000 R CNN
-F 1 "50kΩ" V 2795 3263 50  0000 R CNN
-F 2 "" H 3000 3375 50  0001 C CNN
-F 3 "~" H 3000 3375 50  0001 C CNN
-	1    2750 3450
-	0    1    1    0
-$EndComp
 Wire Wire Line
 	2000 3400 2650 3400
 Wire Wire Line
 	2650 3400 2650 3350
-Wire Wire Line
-	2000 3500 2650 3500
-Wire Wire Line
-	2650 3500 2650 3550
 $Comp
 L power:GND #PWR01
@@
 $EndComp
 Wire Wire Line
-	2150 4100 2150 3300
+	2150 4100 2150 3500
 Wire Wire Line
 	2150 3300 2000 3300
@@
 	6000 4450 6000 4400
 $Comp
-L power:GND #PWR03
-U 1 1 5CAC86AA
-P 2650 4100
-F 0 "#PWR03" H 2650 3850 50  0001 C CNN
-F 1 "GND" H 2655 3927 50  0000 C CNN
-F 2 "" H 2650 4100 50  0001 C CNN
-F 3 "" H 2650 4100 50  0001 C CNN
-	1    2650 4100
-	1    0    0    -1
-$EndComp
-Wire Wire Line
-	2650 4100 2650 3850
-$Comp
 L Device:R_POT RV3
 U 1 1 5CAC9C58
@@
 F 0 "RV3" V 5385 5000 50  0000 C CNN
 F 1 "10kΩ" V 5294 5000 50  0000 C CNN
-F 2 "" H 5500 5000 50  0001 C CNN
+F 2 "Potentiometer_THT:Potentiometer_Piher_PT-10-H01_Horizontal" H 5500 5000 50  0001 C CNN
 F 3 "~" H 5500 5000 50  0001 C CNN
 	1    5500 5000
@@
 F 0 "U3" H 7550 4442 50  0000 C CNN
 F 1 "LM317" H 7550 4351 50  0000 C CNN
-F 2 "" H 7550 4450 50  0001 C CIN
+F 2 "Package_TO_SOT_THT:TO-220-3_Vertical" H 7550 4450 50  0001 C CIN
 F 3 "http://www.ti.com/lit/ds/symlink/lm317.pdf" H 7550 4200 50  0001 C CNN
 	1    7550 4200
@@
 F 0 "R9" H 8370 4496 50  0000 L CNN
 F 1 "1kΩ" H 8370 4405 50  0000 L CNN
-F 2 "" V 8230 4450 50  0001 C CNN
+F 2 "Resistor_THT:R_Axial_DIN0207_L6.3mm_D2.5mm_P10.16mm_Horizontal" V 8230 4450 50  0001 C CNN
 F 3 "~" H 8300 4450 50  0001 C CNN
 	1    8300 4450
@@
 F 0 "C6" H 8068 3896 50  0000 L CNN
 F 1 "470uF" H 8068 3805 50  0000 L CNN
-F 2 "" H 7988 3700 50  0001 C CNN
+F 2 "Capacitor_THT:CP_Radial_D10.0mm_P5.00mm" H 7988 3700 50  0001 C CNN
 F 3 "~" H 7950 3850 50  0001 C CNN
 	1    7950 3850
@@
 F 0 "C4" H 4568 4146 50  0000 L CNN
 F 1 "100uF" H 4568 4055 50  0000 L CNN
-F 2 "" H 4488 3950 50  0001 C CNN
+F 2 "Capacitor_THT:CP_Radial_D8.0mm_P2.50mm" H 4488 3950 50  0001 C CNN
 F 3 "~" H 4450 4100 50  0001 C CNN
 	1    4450 4100
@@
 F 0 "R3" V 3493 4100 50  0000 C CNN
 F 1 "100kΩ" V 3584 4100 50  0000 C CNN
-F 2 "" V 3630 4100 50  0001 C CNN
+F 2 "Resistor_THT:R_Axial_DIN0207_L6.3mm_D2.5mm_P10.16mm_Horizontal" V 3630 4100 50  0001 C CNN
 F 3 "~" H 3700 4100 50  0001 C CNN
 	1    3700 4100
@@
 F 0 "R5" V 3943 4100 50  0000 C CNN
 F 1 "150Ω" V 4034 4100 50  0000 C CNN
-F 2 "" V 4080 4100 50  0001 C CNN
+F 2 "Resistor_THT:R_Axial_DIN0614_L14.3mm_D5.7mm_P5.08mm_Vertical" V 4080 4100 50  0001 C CNN
 F 3 "~" H 4150 4100 50  0001 C CNN
 	1    4150 4100
@@
 F 0 "C3" H 4568 2846 50  0000 L CNN
 F 1 "100uF" H 4568 2755 50  0000 L CNN
-F 2 "" H 4488 2650 50  0001 C CNN
+F 2 "Capacitor_THT:CP_Radial_D8.0mm_P2.50mm" H 4488 2650 50  0001 C CNN
 F 3 "~" H 4450 2800 50  0001 C CNN
 	1    4450 2800
@@
 	2850 3200 3100 3200
 $Comp
-L Device:CP C1
+L Device:C C1
 U 1 1 5CB60F03
 P 3250 3200
 F 0 "C1" V 3505 3200 50  0000 C CNN
 F 1 "2.2uF" V 3414 3200 50  0000 C CNN
-F 2 "" H 3288 3050 50  0001 C CNN
+F 2 "Capacitor_THT:C_Radial_D5.0mm_H11.0mm_P2.00mm" H 3288 3050 50  0001 C CNN
 F 3 "~" H 3250 3200 50  0001 C CNN
 	1    3250 3200
@@
 F 0 "R2" V 3493 2800 50  0000 C CNN
 F 1 "100kΩ" V 3584 2800 50  0000 C CNN
-F 2 "" V 3630 2800 50  0001 C CNN
+F 2 "Resistor_THT:R_Axial_DIN0207_L6.3mm_D2.5mm_P10.16mm_Horizontal" V 3630 2800 50  0001 C CNN
 F 3 "~" H 3700 2800 50  0001 C CNN
 	1    3700 2800
@@
 F 0 "R4" V 3943 2800 50  0000 C CNN
 F 1 "150Ω" V 4034 2800 50  0000 C CNN
-F 2 "" V 4080 2800 50  0001 C CNN
+F 2 "Resistor_THT:R_Axial_DIN0614_L14.3mm_D5.7mm_P5.08mm_Vertical" V 4080 2800 50  0001 C CNN
 F 3 "~" H 4150 2800 50  0001 C CNN
 	1    4150 2800
@@
 $EndComp
 $Comp
-L Device:CP C2
+L Device:C C2
 U 1 1 5CAAFE78
 P 3250 3700
 F 0 "C2" V 3505 3700 50  0000 C CNN
 F 1 "2.2uF" V 3414 3700 50  0000 C CNN
-F 2 "" H 3288 3550 50  0001 C CNN
+F 2 "Capacitor_THT:C_Radial_D5.0mm_H11.0mm_P2.00mm" H 3288 3550 50  0001 C CNN
 F 3 "~" H 3250 3700 50  0001 C CNN
 	1    3250 3700
@@
 F 0 "RV2" V 5385 1950 50  0000 C CNN
 F 1 "10kΩ" V 5294 1950 50  0000 C CNN
-F 2 "" H 5500 1950 50  0001 C CNN
+F 2 "Potentiometer_THT:Potentiometer_Piher_PT-10-H01_Horizontal" H 5500 1950 50  0001 C CNN
 F 3 "~" H 5500 1950 50  0001 C CNN
 	1    5500 1950
@@
 F 0 "R7" H 7970 4496 50  0000 L CNN
 F 1 "10Ω" H 7970 4405 50  0000 L CNN
-F 2 "" V 7830 4450 50  0001 C CNN
+F 2 "Resistor_THT:R_Axial_DIN0207_L6.3mm_D2.5mm_P10.16mm_Horizontal" V 7830 4450 50  0001 C CNN
 F 3 "~" H 7900 4450 50  0001 C CNN
 	1    7900 4450
@@
 F 0 "U2" H 7550 2992 50  0000 C CNN
 F 1 "LM317" H 7550 2901 50  0000 C CNN
-F 2 "" H 7550 3000 50  0001 C CIN
+F 2 "Package_TO_SOT_THT:TO-220-3_Vertical" H 7550 3000 50  0001 C CIN
 F 3 "http://www.ti.com/lit/ds/symlink/lm317.pdf" H 7550 2750 50  0001 C CNN
 	1    7550 2750
@@
 F 0 "R8" H 8370 2546 50  0000 L CNN
 F 1 "1kΩ" H 8370 2455 50  0000 L CNN
-F 2 "" V 8230 2500 50  0001 C CNN
+F 2 "Resistor_THT:R_Axial_DIN0207_L6.3mm_D2.5mm_P10.16mm_Horizontal" V 8230 2500 50  0001 C CNN
 F 3 "~" H 8300 2500 50  0001 C CNN
 	1    8300 2500
@@
 F 0 "C5" H 8068 3146 50  0000 L CNN
 F 1 "470uF" H 8068 3055 50  0000 L CNN
-F 2 "" H 7988 2950 50  0001 C CNN
+F 2 "Capacitor_THT:CP_Radial_D10.0mm_P5.00mm" H 7988 2950 50  0001 C CNN
 F 3 "~" H 7950 3100 50  0001 C CNN
 	1    7950 3100
@@
 F 0 "R6" H 7970 2546 50  0000 L CNN
 F 1 "10Ω" H 7970 2455 50  0000 L CNN
-F 2 "" V 7830 2500 50  0001 C CNN
+F 2 "Resistor_THT:R_Axial_DIN0207_L6.3mm_D2.5mm_P10.16mm_Horizontal" V 7830 2500 50  0001 C CNN
 F 3 "~" H 7900 2500 50  0001 C CNN
 	1    7900 2500
@@
 Wire Wire Line
 	7200 4200 7200 5050
-Wire Wire Line
-	8600 3500 8600 3850
-Wire Wire Line
-	8650 3500 8600 3500
 $Comp
 L power:GND #PWR020
 U 1 1 5CAF0E88
-P 8600 3850
-F 0 "#PWR020" H 8600 3600 50  0001 C CNN
-F 1 "GND" H 8605 3677 50  0000 C CNN
-F 2 "" H 8600 3850 50  0001 C CNN
-F 3 "" H 8600 3850 50  0001 C CNN
-	1    8600 3850
+P 8550 3800
+F 0 "#PWR020" H 8550 3550 50  0001 C CNN
+F 1 "GND" H 8555 3627 50  0000 C CNN
+F 2 "" H 8550 3800 50  0001 C CNN
+F 3 "" H 8550 3800 50  0001 C CNN
+	1    8550 3800
 	1    0    0    -1
 $EndComp
@@
 F 0 "J3" H 8570 3333 50  0000 R CNN
 F 1 "AudioOut" H 8570 3424 50  0000 R CNN
-F 2 "" H 8850 3400 50  0001 C CNN
+F 2 "digikey-footprints:Headphone_Jack_2.5mm_SJ1-3523N" H 8850 3400 50  0001 C CNN
 F 3 "~" H 8850 3400 50  0001 C CNN
 	1    8850 3400
-	-1   0    0    1
-$EndComp
-Wire Wire Line
-	8300 3850 8300 3300
-Wire Wire Line
-	8300 3300 8650 3300
+	-1   0    0    -1
+$EndComp
+Wire Wire Line
+	8300 3850 8300 3500
 Connection ~ 8300 3850
-Wire Wire Line
-	8300 3100 8450 3100
-Wire Wire Line
-	8450 3100 8450 3400
-Wire Wire Line
-	8450 3400 8650 3400
 Connection ~ 8300 3100
 Wire Wire Line
@@
 F 0 "J2" H 1957 7025 50  0000 C CNN
 F 1 "Barrel_Jack" H 1957 6934 50  0000 C CNN
-F 2 "" H 1950 6660 50  0001 C CNN
+F 2 "Connector_BarrelJack:BarrelJack_Horizontal" H 1950 6660 50  0001 C CNN
 F 3 "~" H 1950 6660 50  0001 C CNN
 	1    1900 6700
@@
 F 0 "SW1" H 2700 6835 50  0000 C CNN
 F 1 "SW_SPST" H 2700 6744 50  0000 C CNN
-F 2 "" H 2700 6600 50  0001 C CNN
+F 2 "digikey-footprints:Toggle_Switch_100SP1T1B4M2QE" H 2700 6600 50  0001 C CNN
 F 3 "~" H 2700 6600 50  0001 C CNN
 	1    2700 6600
@@
 F 0 "R1" V 3543 6600 50  0000 C CNN
 F 1 "800Ω" V 3634 6600 50  0000 C CNN
-F 2 "" V 3680 6600 50  0001 C CNN
+F 2 "Resistor_THT:R_Axial_DIN0207_L6.3mm_D2.5mm_P10.16mm_Horizontal" V 3680 6600 50  0001 C CNN
 F 3 "~" H 3750 6600 50  0001 C CNN
 	1    3750 6600
@@
 F 0 "D1" H 4193 6345 50  0000 C CNN
 F 1 "LED" H 4193 6436 50  0000 C CNN
-F 2 "" H 4200 6600 50  0001 C CNN
+F 2 "LED_THT:LED_D5.0mm_Horizontal_O1.27mm_Z3.0mm" H 4200 6600 50  0001 C CNN
 F 3 "~" H 4200 6600 50  0001 C CNN
 	1    4200 6600
@@
 Connection ~ 3050 6600
 Connection ~ 3400 6600
+$Comp
+L Device:R_POT_Dual RV1
+U 1 1 5CAAC98A
+P 2750 3450
+F 0 "RV1" V 2704 3263 50  0000 R CNN
+F 1 "100kΩ" V 2795 3263 50  0000 R CNN
+F 2 "Alps_100KAX2:Alps_100KAX2" H 3000 3375 50  0001 C CNN
+F 3 "~" H 3000 3375 50  0001 C CNN
+	1    2750 3450
+	0    1    1    0
+$EndComp
+Wire Wire Line
+	2650 3550 2650 3500
+Wire Wire Line
+	2650 3500 2150 3500
+Connection ~ 2150 3500
+Wire Wire Line
+	2150 3500 2150 3300
+Wire Wire Line
+	2650 3850 2650 3900
+Wire Wire Line
+	2650 3900 2050 3900
+Wire Wire Line
+	2050 3900 2050 3500
+Wire Wire Line
+	2050 3500 2000 3500
+Wire Wire Line
+	8650 3300 8550 3300
+Wire Wire Line
+	8550 3300 8550 3800
+Wire Wire Line
+	8650 3500 8300 3500
+Wire Wire Line
+	8300 3100 8300 3400
+Wire Wire Line
+	8300 3400 8650 3400
 $EndSCHEMATC

Commit message: fix headphone jack footprint
Parts:
- J1: footprint digikey-footprints:Headphone_Jack_2.5mm_SJ1-3523N -> digikey-footprints:Headphone_Jack_3.5mm_SJ1-3523N
Changed lines of the file:
@@
 EESchema Schematic File Version 4
+LIBS:12AU7-Amplifier-cache
 EELAYER 29 0
 EELAYER END
@@
 F 0 "J1" H 1782 3725 50  0000 C CNN
 F 1 "AudioIn" H 1782 3634 50  0000 C CNN
-F 2 "digikey-footprints:Headphone_Jack_2.5mm_SJ1-3523N" H 1800 3400 50  0001 C CNN
+F 2 "digikey-footprints:Headphone_Jack_3.5mm_SJ1-3523N" H 1800 3400 50  0001 C CNN
 F 3 "~" H 1800 3400 50  0001 C CNN
 	1    1800 3400

Commit message: fix other jack footprint
Parts:
- J3: footprint digikey-footprints:Headphone_Jack_2.5mm_SJ1-3523N -> digikey-footprints:Headphone_Jack_3.5mm_SJ1-3523N
Changed lines of the file:
@@
 F 0 "J3" H 8570 3333 50  0000 R CNN
 F 1 "AudioOut" H 8570 3424 50  0000 R CNN
-F 2 "digikey-footprints:Headphone_Jack_2.5mm_SJ1-3523N" H 8850 3400 50  0001 C CNN
+F 2 "digikey-footprints:Headphone_Jack_3.5mm_SJ1-3523N" H 8850 3400 50  0001 C CNN
 F 3 "~" H 8850 3400 50  0001 C CNN
 	1    8850 3400

Commit message: PCB footprint placement
Parts:
- removed J1: AudioIn, digikey-footprints:Headphone_Jack_3.5mm_SJ1-3523N, symbol Connector:AudioJack3
- removed J3: AudioOut, digikey-footprints:Headphone_Jack_3.5mm_SJ1-3523N, symbol Connector:AudioJack3
- added CON1: AudioIn, digikey-footprints:Headphone_Jack_3.5mm_SJ1-3523N, symbol dk_Barrel-Audio-Connectors:SJ1-3523N
- added CON2: AudioOut, digikey-footprints:Headphone_Jack_3.5mm_SJ1-3523N, symbol dk_Barrel-Audio-Connectors:SJ1-3523N
- U1: footprint Valve:Valve_Noval_P -> 12AU7:12AU7
- renumbered J2 to J1, R2 to R1, R3 to R2, R1 to R3
Changed lines of the file:
@@
 Comment4 ""
 $EndDescr
-$Comp
-L Connector:AudioJack3 J1
-U 1 1 5CAA7597
-P 1800 3400
-F 0 "J1" H 1782 3725 50  0000 C CNN
-F 1 "AudioIn" H 1782 3634 50  0000 C CNN
-F 2 "digikey-footprints:Headphone_Jack_3.5mm_SJ1-3523N" H 1800 3400 50  0001 C CNN
-F 3 "~" H 1800 3400 50  0001 C CNN
-	1    1800 3400
-	1    0    0    -1
-$EndComp
-Wire Wire Line
-	2000 3400 2650 3400
 Wire Wire Line
 	2650 3400 2650 3350
@@
 $EndComp
 Wire Wire Line
-	2150 4100 2150 3500
-Wire Wire Line
-	2150 3300 2000 3300
+	2150 4100 2150 3600
 $Comp
 L Valve:ECC81 U1
@@
 F 0 "U1" V 5954 3778 50  0000 L CNN
 F 1 "12AU7" V 6045 3778 50  0000 L CNN
-F 2 "Valve:Valve_Noval_P" H 6270 3050 50  0001 C CNN
+F 2 "12AU7:12AU7" H 6270 3050 50  0001 C CNN
 F 3 "http://www.r-type.org/pdfs/ecc81.pdf" H 6000 3450 50  0001 C CNN
 	3    6000 3450
@@
 F 0 "U1" V 6273 2850 50  0000 C CNN
 F 1 "12AU7" V 6364 2850 50  0000 C CNN
-F 2 "Valve:Valve_Noval_P" H 6270 2450 50  0001 C CNN
+F 2 "12AU7:12AU7" H 6270 2450 50  0001 C CNN
 F 3 "http://www.r-type.org/pdfs/ecc81.pdf" H 6000 2850 50  0001 C CNN
 	2    6000 2850
@@
 	2850 3700 3100 3700
 $Comp
-L Device:R R3
+L Device:R R2
 U 1 1 5CAA5F31
 P 3700 4100
-F 0 "R3" V 3493 4100 50  0000 C CNN
+F 0 "R2" V 3493 4100 50  0000 C CNN
 F 1 "100kΩ" V 3584 4100 50  0000 C CNN
 F 2 "Resistor_THT:R_Axial_DIN0207_L6.3mm_D2.5mm_P10.16mm_Horizontal" V 3630 4100 50  0001 C CNN
@@
 $EndComp
 $Comp
-L Device:R R2
+L Device:R R1
 U 1 1 5CB60F09
 P 3700 2800
-F 0 "R2" V 3493 2800 50  0000 C CNN
+F 0 "R1" V 3493 2800 50  0000 C CNN
 F 1 "100kΩ" V 3584 2800 50  0000 C CNN
 F 2 "Resistor_THT:R_Axial_DIN0207_L6.3mm_D2.5mm_P10.16mm_Horizontal" V 3630 2800 50  0001 C CNN
@@
 F 0 "U1" V 6365 4100 50  0000 C CNN
 F 1 "12AU7" V 6274 4100 50  0000 C CNN
-F 2 "Valve:Valve_Noval_P" H 6270 3700 50  0001 C CNN
+F 2 "12AU7:12AU7" H 6270 3700 50  0001 C CNN
 F 3 "http://www.r-type.org/pdfs/ecc81.pdf" H 6000 4100 50  0001 C CNN
 	1    6000 4100
@@
 L power:GND #PWR020
 U 1 1 5CAF0E88
-P 8550 3800
-F 0 "#PWR020" H 8550 3550 50  0001 C CNN
-F 1 "GND" H 8555 3627 50  0000 C CNN
-F 2 "" H 8550 3800 50  0001 C CNN
-F 3 "" H 8550 3800 50  0001 C CNN
-	1    8550 3800
-	1    0    0    -1
-$EndComp
-$Comp
-L Connector:AudioJack3 J3
-U 1 1 5CAEEF58
-P 8850 3400
-F 0 "J3" H 8570 3333 50  0000 R CNN
-F 1 "AudioOut" H 8570 3424 50  0000 R CNN
-F 2 "digikey-footprints:Headphone_Jack_3.5mm_SJ1-3523N" H 8850 3400 50  0001 C CNN
-F 3 "~" H 8850 3400 50  0001 C CNN
-	1    8850 3400
-	-1   0    0    -1
+P 8500 3850
+F 0 "#PWR020" H 8500 3600 50  0001 C CNN
+F 1 "GND" H 8505 3677 50  0000 C CNN
+F 2 "" H 8500 3850 50  0001 C CNN
+F 3 "" H 8500 3850 50  0001 C CNN
+	1    8500 3850
+	1    0    0    -1
 $EndComp
 Wire Wire Line
@@
 	4950 3800 4950 4550
 $Comp
-L Connector:Barrel_Jack J2
+L Connector:Barrel_Jack J1
 U 1 1 5CC919F9
 P 1900 6700
-F 0 "J2" H 1957 7025 50  0000 C CNN
+F 0 "J1" H 1957 7025 50  0000 C CNN
 F 1 "Barrel_Jack" H 1957 6934 50  0000 C CNN
 F 2 "Connector_BarrelJack:BarrelJack_Horizontal" H 1950 6660 50  0001 C CNN
@@
 	2200 6600 2500 6600
 $Comp
-L Device:R R1
+L Device:R R3
 U 1 1 5CC9A575
 P 3750 6600
-F 0 "R1" V 3543 6600 50  0000 C CNN
+F 0 "R3" V 3543 6600 50  0000 C CNN
 F 1 "800Ω" V 3634 6600 50  0000 C CNN
 F 2 "Resistor_THT:R_Axial_DIN0207_L6.3mm_D2.5mm_P10.16mm_Horizontal" V 3680 6600 50  0001 C CNN
@@
 	4500 6600 4500 6900
 $Comp
-L power:PWR_FLAG #FLG0101
+L power:PWR_FLAG #FLG02
 U 1 1 5CD1CF3B
 P 3400 6400
-F 0 "#FLG0101" H 3400 6475 50  0001 C CNN
+F 0 "#FLG02" H 3400 6475 50  0001 C CNN
 F 1 "PWR_FLAG" H 3400 6573 50  0000 C CNN
 F 2 "" H 3400 6400 50  0001 C CNN
@@
 $EndComp
 $Comp
-L power:GND #PWR0101
+L power:GND #PWR03
 U 1 1 5CD310AE
 P 2650 2800
-F 0 "#PWR0101" H 2650 2550 50  0001 C CNN
+F 0 "#PWR03" H 2650 2550 50  0001 C CNN
 F 1 "GND" H 2655 2627 50  0000 C CNN
 F 2 "" H 2650 2800 50  0001 C CNN
@@
 	2650 2800 2650 3050
 $Comp
-L power:PWR_FLAG #FLG0102
+L power:PWR_FLAG #FLG01
 U 1 1 5CD351E6
 P 2700 6900
-F 0 "#FLG0102" H 2700 6975 50  0001 C CNN
+F 0 "#FLG01" H 2700 6975 50  0001 C CNN
 F 1 "PWR_FLAG" H 2700 7073 50  0000 C CNN
 F 2 "" H 2700 6900 50  0001 C CNN
@@
 Wire Wire Line
 	2650 3500 2150 3500
-Connection ~ 2150 3500
-Wire Wire Line
-	2150 3500 2150 3300
 Wire Wire Line
 	2650 3850 2650 3900
@@
 	2650 3900 2050 3900
 Wire Wire Line
+	8600 3600 8500 3600
+Wire Wire Line
+	8500 3600 8500 3850
+Wire Wire Line
+	8300 3100 8300 3400
+$Comp
+L dk_Barrel-Audio-Connectors:SJ1-3523N CON1
+U 1 1 5CAC6A75
+P 1550 3500
+F 0 "CON1" H 1608 3887 60  0000 C CNN
+F 1 "AudioIn" H 1608 3781 60  0000 C CNN
+F 2 "digikey-footprints:Headphone_Jack_3.5mm_SJ1-3523N" H 1750 3700 60  0001 L CNN
+F 3 "https://www.cui.com/product/resource/digikeypdf/sj1-352xn_series.pdf" H 1750 3800 60  0001 L CNN
+F 4 "CP1-3523N-ND" H 1750 3900 60  0001 L CNN "Digi-Key_PN"
+F 5 "SJ1-3523N" H 1750 4000 60  0001 L CNN "MPN"
+F 6 "Connectors, Interconnects" H 1750 4100 60  0001 L CNN "Category"
+F 7 "Barrel - Audio Connectors" H 1750 4200 60  0001 L CNN "Family"
+F 8 "https://www.cui.com/product/resource/digikeypdf/sj1-352xn_series.pdf" H 1750 4300 60  0001 L CNN "DK_Datasheet_Link"
+F 9 "/product-detail/en/cui-inc/SJ1-3523N/CP1-3523N-ND/738689" H 1750 4400 60  0001 L CNN "DK_Detail_Page"
+F 10 "CONN JACK STEREO 3.5MM R/A" H 1750 4500 60  0001 L CNN "Description"
+F 11 "CUI Inc." H 1750 4600 60  0001 L CNN "Manufacturer"
+F 12 "Active" H 1750 4700 60  0001 L CNN "Status"
+	1    1550 3500
+	1    0    0    -1
+$EndComp
+Wire Wire Line
+	1950 3400 2650 3400
+Wire Wire Line
+	1950 3600 2150 3600
+Connection ~ 2150 3600
+Wire Wire Line
+	2150 3600 2150 3500
+Wire Wire Line
 	2050 3900 2050 3500
 Wire Wire Line
-	2050 3500 2000 3500
-Wire Wire Line
-	8650 3300 8550 3300
-Wire Wire Line
-	8550 3300 8550 3800
-Wire Wire Line
-	8650 3500 8300 3500
-Wire Wire Line
-	8300 3100 8300 3400
-Wire Wire Line
-	8300 3400 8650 3400
+	2050 3500 1950 3500
+$Comp
+L dk_Barrel-Audio-Connectors:SJ1-3523N CON2
+U 1 1 5CB0F07A
+P 9000 3500
+F 0 "CON2" H 8672 3553 60  0000 R CNN
+F 1 "AudioOut" H 8672 3447 60  0000 R CNN
+F 2 "digikey-footprints:Headphone_Jack_3.5mm_SJ1-3523N" H 9200 3700 60  0001 L CNN
+F 3 "https://www.cui.com/product/resource/digikeypdf/sj1-352xn_series.pdf" H 9200 3800 60  0001 L CNN
+F 4 "CP1-3523N-ND" H 9200 3900 60  0001 L CNN "Digi-Key_PN"
+F 5 "SJ1-3523N" H 9200 4000 60  0001 L CNN "MPN"
+F 6 "Connectors, Interconnects" H 9200 4100 60  0001 L CNN "Category"
+F 7 "Barrel - Audio Connectors" H 9200 4200 60  0001 L CNN "Family"
+F 8 "https://www.cui.com/product/resource/digikeypdf/sj1-352xn_series.pdf" H 9200 4300 60  0001 L CNN "DK_Datasheet_Link"
+F 9 "/product-detail/en/cui-inc/SJ1-3523N/CP1-3523N-ND/738689" H 9200 4400 60  0001 L CNN "DK_Detail_Page"
+F 10 "CONN JACK STEREO 3.5MM R/A" H 9200 4500 60  0001 L CNN "Description"
+F 11 "CUI Inc." H 9200 4600 60  0001 L CNN "Manufacturer"
+F 12 "Active" H 9200 4700 60  0001 L CNN "Status"
+	1    9000 3500
+	-1   0    0    -1
+$EndComp
+Wire Wire Line
+	8300 3400 8600 3400
+Wire Wire Line
+	8300 3500 8600 3500
 $EndSCHEMATC

Commit message: Add ground plane and trace routing
Parts:
- J1: symbol Connector:Barrel_Jack -> Connector:Barrel_Jack_Switch
Connections:
- wire segments 121 -> 123
Changed lines of the file:
@@
 	4950 3800 4950 4550
 $Comp
-L Connector:Barrel_Jack J1
+L Connector:Barrel_Jack_Switch J1
 U 1 1 5CC919F9
 P 1900 6700
@@
 Wire Wire Line
 	8300 3500 8600 3500
+Wire Wire Line
+	2200 6700 2400 6700
+Wire Wire Line
+	2400 6700 2400 6800
 $EndSCHEMATC
