File: 12AU7-Amplifier.sch (KiCad schematic (older format))
At the start: 28 parts, among them CON1 AudioIn, CON2 AudioOut, J1 Barrel_Jack, Q1 IRF510, Q2 IRF510, SW1 SW_SPST, U1 12AU7, U2 LM317, U3 LM317

Commit message: add smoothing capacitor
Parts:
- added C7: 10uF, Capacitor_THT:CP_Radial_D5.0mm_P2.50mm, symbol Device:CP
Connections:
- wire segments 123 -> 126
Other:
- moved on the sheet: D1, J1, R3
Changed lines of the file:
@@
 L Connector:Barrel_Jack_Switch J1
 U 1 1 5CC919F9
-P 1900 6700
-F 0 "J1" H 1957 7025 50  0000 C CNN
-F 1 "Barrel_Jack" H 1957 6934 50  0000 C CNN
-F 2 "Connector_BarrelJack:BarrelJack_Horizontal" H 1950 6660 50  0001 C CNN
-F 3 "~" H 1950 6660 50  0001 C CNN
-	1    1900 6700
+P 1950 6300
+F 0 "J1" H 2007 6625 50  0000 C CNN
+F 1 "Barrel_Jack" H 2007 6534 50  0000 C CNN
+F 2 "Connector_BarrelJack:BarrelJack_Horizontal" H 2000 6260 50  0001 C CNN
+F 3 "~" H 2000 6260 50  0001 C CNN
+	1    1950 6300
 	1    0    0    -1
 $EndComp
@@
 L power:GND #PWR02
 U 1 1 5CC923DC
-P 2400 6900
-F 0 "#PWR02" H 2400 6650 50  0001 C CNN
-F 1 "GND" H 2405 6727 50  0000 C CNN
-F 2 "" H 2400 6900 50  0001 C CNN
-F 3 "" H 2400 6900 50  0001 C CNN
-	1    2400 6900
-	-1   0    0    -1
-$EndComp
-Wire Wire Line
-	2400 6900 2400 6800
-Wire Wire Line
-	2400 6800 2200 6800
+P 2450 6700
+F 0 "#PWR02" H 2450 6450 50  0001 C CNN
+F 1 "GND" H 2455 6527 50  0000 C CNN
+F 2 "" H 2450 6700 50  0001 C CNN
+F 3 "" H 2450 6700 50  0001 C CNN
+	1    2450 6700
+	-1   0    0    -1
+$EndComp
+Wire Wire Line
+	2450 6700 2450 6400
+Wire Wire Line
+	2450 6400 2250 6400
 $Comp
 L Switch:SW_SPST SW1
 U 1 1 5CC9635A
-P 2700 6600
-F 0 "SW1" H 2700 6835 50  0000 C CNN
-F 1 "SW_SPST" H 2700 6744 50  0000 C CNN
-F 2 "digikey-footprints:Toggle_Switch_100SP1T1B4M2QE" H 2700 6600 50  0001 C CNN
-F 3 "~" H 2700 6600 50  0001 C CNN
-	1    2700 6600
-	1    0    0    -1
-$EndComp
-Wire Wire Line
-	2200 6600 2500 6600
+P 2900 6200
+F 0 "SW1" H 2900 6435 50  0000 C CNN
+F 1 "SW_SPST" H 2900 6344 50  0000 C CNN
+F 2 "digikey-footprints:Toggle_Switch_100SP1T1B4M2QE" H 2900 6200 50  0001 C CNN
+F 3 "~" H 2900 6200 50  0001 C CNN
+	1    2900 6200
+	1    0    0    -1
+$EndComp
+Wire Wire Line
+	2250 6200 2700 6200
 $Comp
 L Device:R R3
 U 1 1 5CC9A575
-P 3750 6600
-F 0 "R3" V 3543 6600 50  0000 C CNN
-F 1 "800Ω" V 3634 6600 50  0000 C CNN
-F 2 "Resistor_THT:R_Axial_DIN0207_L6.3mm_D2.5mm_P10.16mm_Horizontal" V 3680 6600 50  0001 C CNN
-F 3 "~" H 3750 6600 50  0001 C CNN
-	1    3750 6600
+P 4400 6200
+F 0 "R3" V 4193 6200 50  0000 C CNN
+F 1 "800Ω" V 4284 6200 50  0000 C CNN
+F 2 "Resistor_THT:R_Axial_DIN0207_L6.3mm_D2.5mm_P10.16mm_Horizontal" V 4330 6200 50  0001 C CNN
+F 3 "~" H 4400 6200 50  0001 C CNN
+	1    4400 6200
 	0    -1   1    0
 $EndComp
@@
 L power:+12V #PWR04
 U 1 1 5CCB4117
-P 3050 6400
-F 0 "#PWR04" H 3050 6250 50  0001 C CNN
-F 1 "+12V" H 3065 6573 50  0000 C CNN
-F 2 "" H 3050 6400 50  0001 C CNN
-F 3 "" H 3050 6400 50  0001 C CNN
-	1    3050 6400
-	1    0    0    -1
-$EndComp
-Wire Wire Line
-	3050 6400 3050 6600
-Wire Wire Line
-	3050 6600 2900 6600
-Wire Wire Line
-	3400 6600 3600 6600
+P 3700 6000
+F 0 "#PWR04" H 3700 5850 50  0001 C CNN
+F 1 "+12V" H 3715 6173 50  0000 C CNN
+F 2 "" H 3700 6000 50  0001 C CNN
+F 3 "" H 3700 6000 50  0001 C CNN
+	1    3700 6000
+	1    0    0    -1
+$EndComp
+Wire Wire Line
+	3700 6000 3700 6200
+Wire Wire Line
+	4050 6200 4250 6200
 $Comp
 L Device:LED D1
 U 1 1 5CCBBC9F
-P 4200 6600
-F 0 "D1" H 4193 6345 50  0000 C CNN
-F 1 "LED" H 4193 6436 50  0000 C CNN
-F 2 "LED_THT:LED_D5.0mm_Horizontal_O1.27mm_Z3.0mm" H 4200 6600 50  0001 C CNN
-F 3 "~" H 4200 6600 50  0001 C CNN
-	1    4200 6600
+P 4850 6200
+F 0 "D1" H 4843 5945 50  0000 C CNN
+F 1 "LED" H 4843 6036 50  0000 C CNN
+F 2 "LED_THT:LED_D5.0mm_Horizontal_O1.27mm_Z3.0mm" H 4850 6200 50  0001 C CNN
+F 3 "~" H 4850 6200 50  0001 C CNN
+	1    4850 6200
 	-1   0    0    1
 $EndComp
 Wire Wire Line
-	3900 6600 4050 6600
+	4550 6200 4700 6200
 $Comp
 L power:GND #PWR09
 U 1 1 5CCC0B1A
-P 4500 6900
-F 0 "#PWR09" H 4500 6650 50  0001 C CNN
-F 1 "GND" H 4505 6727 50  0000 C CNN
-F 2 "" H 4500 6900 50  0001 C CNN
-F 3 "" H 4500 6900 50  0001 C CNN
-	1    4500 6900
-	-1   0    0    -1
-$EndComp
-Wire Wire Line
-	4350 6600 4500 6600
-Wire Wire Line
-	4500 6600 4500 6900
+P 5150 6700
+F 0 "#PWR09" H 5150 6450 50  0001 C CNN
+F 1 "GND" H 5155 6527 50  0000 C CNN
+F 2 "" H 5150 6700 50  0001 C CNN
+F 3 "" H 5150 6700 50  0001 C CNN
+	1    5150 6700
+	-1   0    0    -1
+$EndComp
+Wire Wire Line
+	5000 6200 5150 6200
+Wire Wire Line
+	5150 6200 5150 6700
 $Comp
 L power:PWR_FLAG #FLG02
 U 1 1 5CD1CF3B
-P 3400 6400
-F 0 "#FLG02" H 3400 6475 50  0001 C CNN
-F 1 "PWR_FLAG" H 3400 6573 50  0000 C CNN
-F 2 "" H 3400 6400 50  0001 C CNN
-F 3 "~" H 3400 6400 50  0001 C CNN
-	1    3400 6400
+P 4050 6000
+F 0 "#FLG02" H 4050 6075 50  0001 C CNN
+F 1 "PWR_FLAG" H 4050 6173 50  0000 C CNN
+F 2 "" H 4050 6000 50  0001 C CNN
+F 3 "~" H 4050 6000 50  0001 C CNN
+	1    4050 6000
 	1    0    0    -1
 $EndComp
@@
 L power:PWR_FLAG #FLG01
 U 1 1 5CD351E6
-P 2700 6900
-F 0 "#FLG01" H 2700 6975 50  0001 C CNN
-F 1 "PWR_FLAG" H 2700 7073 50  0000 C CNN
-F 2 "" H 2700 6900 50  0001 C CNN
-F 3 "~" H 2700 6900 50  0001 C CNN
-	1    2700 6900
+P 2750 6700
+F 0 "#FLG01" H 2750 6775 50  0001 C CNN
+F 1 "PWR_FLAG" H 2750 6873 50  0000 C CNN
+F 2 "" H 2750 6700 50  0001 C CNN
+F 3 "~" H 2750 6700 50  0001 C CNN
+	1    2750 6700
 	-1   0    0    1
 $EndComp
 Wire Wire Line
-	2700 6900 2700 6800
-Wire Wire Line
-	2700 6800 2400 6800
-Connection ~ 2400 6800
-Wire Wire Line
-	3400 6400 3400 6600
-Wire Wire Line
-	3050 6600 3400 6600
-Connection ~ 3050 6600
-Connection ~ 3400 6600
+	2750 6700 2750 6400
+Wire Wire Line
+	2750 6400 2450 6400
+Connection ~ 2450 6400
+Wire Wire Line
+	4050 6000 4050 6200
+Wire Wire Line
+	3700 6200 4050 6200
+Connection ~ 3700 6200
+Connection ~ 4050 6200
 $Comp
 L Device:R_POT_Dual RV1
@@
 	8300 3500 8600 3500
 Wire Wire Line
-	2200 6700 2400 6700
-Wire Wire Line
-	2400 6700 2400 6800
+	2250 6300 2450 6300
+Wire Wire Line
+	2450 6300 2450 6400
+Wire Wire Line
+	3700 6200 3350 6200
+$Comp
+L Device:CP C7
+U 1 1 5CB59ACC
+P 3350 6450
+F 0 "C7" H 3468 6496 50  0000 L CNN
+F 1 "10uF" H 3468 6405 50  0000 L CNN
+F 2 "Capacitor_THT:CP_Radial_D5.0mm_P2.50mm" H 3388 6300 50  0001 C CNN
+F 3 "~" H 3350 6450 50  0001 C CNN
+	1    3350 6450
+	1    0    0    -1
+$EndComp
+Wire Wire Line
+	3350 6300 3350 6200
+Connection ~ 3350 6200
+Wire Wire Line
+	3350 6200 3100 6200
+$Comp
+L power:GND #PWR021
+U 1 1 5CB85CDE
+P 3350 6700
+F 0 "#PWR021" H 3350 6450 50  0001 C CNN
+F 1 "GND" H 3355 6527 50  0000 C CNN
+F 2 "" H 3350 6700 50  0001 C CNN
+F 3 "" H 3350 6700 50  0001 C CNN
+	1    3350 6700
+	-1   0    0    -1
+$EndComp
+Wire Wire Line
+	3350 6700 3350 6600
 $EndSCHEMATC

Commit message: reroute and final
Parts:
- removed SW1: SW_SPST, digikey-footprints:Toggle_Switch_100SP1T1B4M2QE, symbol Switch:SW_SPST
- added SW1: SW_SPDT, Switch_200MSP1T1B2M6QE:Switch_SPDT, symbol Switch:SW_SPDT
Connections:
- wire segments 126 -> 128
- no-connect marks 0 -> 1
Changed lines of the file:
@@
 Wire Wire Line
 	2450 6400 2250 6400
-$Comp
-L Switch:SW_SPST SW1
-U 1 1 5CC9635A
-P 2900 6200
-F 0 "SW1" H 2900 6435 50  0000 C CNN
-F 1 "SW_SPST" H 2900 6344 50  0000 C CNN
-F 2 "digikey-footprints:Toggle_Switch_100SP1T1B4M2QE" H 2900 6200 50  0001 C CNN
-F 3 "~" H 2900 6200 50  0001 C CNN
-	1    2900 6200
-	1    0    0    -1
-$EndComp
-Wire Wire Line
-	2250 6200 2700 6200
+Wire Wire Line
+	2250 6200 2550 6200
 $Comp
 L Device:R R3
@@
 Wire Wire Line
 	3350 6700 3350 6600
+$Comp
+L Switch:SW_SPDT SW1
+U 1 1 5CB5A4D3
+P 2750 6200
+F 0 "SW1" H 2750 6485 50  0000 C CNN
+F 1 "SW_SPDT" H 2750 6394 50  0000 C CNN
+F 2 "Switch_200MSP1T1B2M6QE:Switch_SPDT" H 2750 6200 50  0001 C CNN
+F 3 "~" H 2750 6200 50  0001 C CNN
+	1    2750 6200
+	1    0    0    -1
+$EndComp
+Wire Wire Line
+	2950 6300 3100 6300
+Wire Wire Line
+	3100 6300 3100 6200
+NoConn ~ 2950 6100
 $EndSCHEMATC
