File: 12AU7-Amplifier.kicad_pcb (KiCad board)
At the start: 4 copper layers, 75 x 120 mm, 43 parts, among them J1 SJ1-3523N, J2 Barrel_Jack, J3 SJ1-3523N, Q1 IRF510, Q2 IRF510, SW1 100SP1T2B4M7QE, U1 12AU7, U2 LM317, U3 LM317

Commit message: Trace layout, silkscreen, assembly model
Parts:
- moved R7 36.9 mm to (127.7, 96.0), turned to 180 degrees
- moved R3 36.0 mm to (127.5, 60.5)
- moved R4 36.0 mm to (117.5, 55.5)
- moved R6 35.5 mm to (117.5, 91.0)
- moved C11 5.50 mm to (129.0, 102.0), turned to 270 degrees
- moved C8 5.50 mm to (116.0, 102.0), turned to 270 degrees
Routing:
- net Net-(J2-Pad1): track 0.00 -> 132.2 mm
- net Net-(C8-Pad2): track 0.00 -> 97.5 mm
- net Net-(C10-Pad1): track 0.00 -> 91.4 mm
- net Net-(C8-Pad1): track 0.00 -> 76.9 mm
- net Net-(C10-Pad2): track 0.00 -> 55.8 mm
- net Net-(C1-Pad1): track 0.00 -> 55.1 mm
- net Net-(Q2-Pad1): track 0.00 -> 53.2 mm
- net Net-(C2-Pad1): track 0.00 -> 49.5 mm
- net Net-(Q1-Pad1): track 0.00 -> 45.3 mm
- net Net-(C4-Pad1): track 0.00 -> 44.8 mm
- net Net-(C5-Pad1): track 0.00 -> 44.6 mm
- net Net-(J1-Pad3): track 0.00 -> 39.2 mm
- net Net-(C2-Pad2): track 0.03 -> 37.3 mm
- net Net-(C1-Pad2): track 0.00 -> 23.4 mm
- net Net-(J1-Pad2): track 0.00 -> 22.5 mm
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Other:
- board text added: "12AU7 AMPLIFIER"
- board text added: "Aaron & Ryan Shappell"
