File: 12AU7-Amplifier.kicad_pcb (KiCad board)
At the start: 4 copper layers, 75 x 120 mm, 43 parts, among them J1 SJ1-3523N, J2 Barrel_Jack, J3 SJ1-3523N, Q1 IRF510, Q2 IRF510, SW1 100SP1T2B4M7QE, U1 12AU7, U2 LM317, U3 LM317

Commit message: Stupid mistake...
Routing:
- removed copper zone on PWR.Cu, net GND

Commit message: Convert to kicad 6
Routing:
- added copper zone on In1.Cu, net +12V
- added copper zone on In2.Cu, net GND
- removed copper zone on PWR.Cu, net +12V
- removed copper zone on GND.Cu, net GND
Other:
- net class Default removed
